File: V2/PCB/ArduinoNano33Proto-V2.0.brd (EAGLE design)
At the start: 100 x 46 mm, 53 parts, among them J1 RJ11, J2 RJ11, J23 455-1750-1-ND, J24 455-1750-1-ND, J26 455-1750-1-ND, J27 455-1750-1-ND, J31 455-1750-1-ND, J32 455-1750-1-ND, J38 455-1750-1-ND, J39 455-1750-1-ND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

Commit message: Update to V2 (RJ11) board.
Parts:
- added J11, J21: (no value), SparkFun-Connectors:1X16_NO_SILK
- moved J1 2.22 mm to (95.0, 31.0)
- moved J2 2.22 mm to (95.0, 15.0)
- moved J3 2.22 mm to (82.5, 25.4)
- moved J4 2.22 mm to (82.5, 7.62)
